File: hardware/pcb/fercus-right/fercus-right.kicad_sch (KiCad schematic)
At the start: 274 parts, among them J1 USB_C_Receptacle_USB2.0, J2 USB_C_Receptacle_USB2.0, J3 Conn_01x06_MountingPin, J5 Conn_01x03, Q1 BSS138, Q10 BSS138, Q2 BSS138, Q3 BSS138, Q4 BSS138, Q5 BSS138, Q6 BSS138, Q7 BSS138, Q8 BSS138, Q9 BSS138, SW1 SW_Push, SW2 SW_Push, SW3 SW_Push, SW4 SW_Push, SW6 SW_Push, SW7 SW_SPDT, SW8 SW_Push, U1 XC6206P332MR, U2 CH32V208CBU6, U3 ETA9084E10, Y1 32MHz, CL12pF, Y2 32.768kHz, CL12.5pF

Commit message: merge
    fw:
    - fix usb product string, vid
    - add rf_phy_hop
    - add RF_BondingErase()
    - change default layout key fn to pause
    - fix power manager poweroff when usb disconnect
    - add usb compatibility interface

    hw:
    - change eta9084 iset resistor footprint to 0402
    - change fpc connector part
    - fix ir resistor value
    - change pcb thinkness to 1.6mm
    - fix footprint of pt and ir
    - fix rf ant trace
    - fix usb trace
    - add fercus-dongle-usb-c

    doc:
    - fix layout
    - add manual
Parts:
- AE1: footprint chulaine:ANT-F-1-2.4G-1.2MM-FR4-WCH_Right_NoMask -> wch-ant:WCH_MIFA-1_2.4GHz_1.6mm_FR4_Right_NoMask
- IR1, IR10, IR11, IR12, IR13, IR14, IR15, IR16, IR17, IR18, IR19, IR2, IR20, IR21, IR22, IR23, IR24, IR25, IR26, IR27, IR28, IR29, IR3, IR30, IR31, IR32, IR33, IR34, IR35, IR36, IR37, IR38, IR39, IR4, IR40, IR41, IR42, IR5, IR6, IR7, IR8, IR9: value IR -> KTR-0602IRC-850
- J3: value Conn_01x06_MountingPin -> AFH34-S06FIA-1H
- PT1, PT10, PT11, PT12, PT13, PT14, PT15, PT16, PT17, PT18, PT19, PT2, PT20, PT21, PT22, PT23, PT24, PT25, PT26, PT27, PT28, PT29, PT3, PT30, PT31, PT32, PT33, PT34, PT35, PT36, PT37, PT38, PT39, PT4, PT40, PT41, PT42, PT5, PT6, PT7, PT8, PT9: value Q_Photo_NPN_EC -> KTR-0602PTD
- R37: footprint Resistor_SMD:R_0603_1608Metric -> Resistor_SMD:R_0402_1005Metric
- TP2: now not fitted; now left out of the parts list
Connections:
- net usart1_tx: now also J1.A8 (SBU1)
- no-connect marks 9 -> 7

Commit message: merge
hw:
- fix sch
- fix plate
- rename to fercus-dongle-usb-a

doc:
- add assembly
Parts:
- removed C17, C21, C27, C28, C29, C30: 100nF, Capacitor_SMD:C_0603_1608Metric, symbol Device:C
- added C39, C40, C41, C42, C43, C44: 100nF, Capacitor_SMD:C_0603_1608Metric, symbol Device:C
- added TP3: TestPoint, TestPoint:TestPoint_Pad_D1.0mm, symbol Connector:TestPoint
- AE1: footprint wch-ant:WCH_MIFA-1_2.4GHz_1.6mm_FR4_Right_NoMask -> wch-ant:WCH_MIFA-1_2.4GHz_1.6mm_FR4_Right
- J5: value Conn_01x03 -> Molex_PicoBlade_53261-0371_1x03-1MP_P1.25mm_Horizontal
- SW1: renamed from SWO1; value SW_LPO -> SW_Optical
- SW10: renamed from SWO10; value SW_LPO -> SW_Optical
- SW11: renamed from SWO11; value SW_LPO -> SW_Optical
- SW12: renamed from SWO12; value SW_LPO -> SW_Optical
- SW13: renamed from SWO13; value SW_LPO -> SW_Optical
- SW14: renamed from SWO14; value SW_LPO -> SW_Optical
- SW15: renamed from SWO15; value SW_LPO -> SW_Optical
- SW16: renamed from SWO16; value SW_LPO -> SW_Optical
- SW17: renamed from SWO17; value SW_LPO -> SW_Optical
- SW18: renamed from SWO18; value SW_LPO -> SW_Optical
- SW19: renamed from SWO19; value SW_LPO -> SW_Optical
- SW2: renamed from SWO2; value SW_LPO -> SW_Optical
- SW20: renamed from SWO20; value SW_LPO -> SW_Optical
- SW21: renamed from SWO21; value SW_LPO -> SW_Optical
- SW22: renamed from SWO22; value SW_LPO -> SW_Optical
- SW23: renamed from SWO23; value SW_LPO -> SW_Optical
- SW24: renamed from SWO24; value SW_LPO -> SW_Optical
- SW25: renamed from SWO25; value SW_LPO -> SW_Optical
- SW26: renamed from SWO26; value SW_LPO -> SW_Optical
- SW27: renamed from SWO27; value SW_LPO -> SW_Optical
- SW28: renamed from SWO28; value SW_LPO -> SW_Optical
- SW29: renamed from SWO29; value SW_LPO -> SW_Optical
- SW3: renamed from SWO3; value SW_LPO -> SW_Optical
- SW30: renamed from SWO30; value SW_LPO -> SW_Optical
- SW31: renamed from SWO31; value SW_LPO -> SW_Optical
- SW32: renamed from SWO32; value SW_LPO -> SW_Optical
- SW33: renamed from SWO33; value SW_LPO -> SW_Optical
- SW34: renamed from SWO34; value SW_LPO -> SW_Optical
- SW35: renamed from SWO35; value SW_LPO -> SW_Optical
- SW36: renamed from SWO36; value SW_LPO -> SW_Optical
- SW37: renamed from SWO37; value SW_LPO -> SW_Optical
- SW38: renamed from SWO38; value SW_LPO -> SW_Optical
- SW39: renamed from SWO39; value SW_LPO -> SW_Optical
- SW4: renamed from SWO4; value SW_LPO -> SW_Optical
- SW40: renamed from SWO40; value SW_LPO -> SW_Optical
- SW41: renamed from SWO41; value SW_LPO -> SW_Optical
- SW42: renamed from SWO42; value SW_LPO -> SW_Optical
- SW5: renamed from SWO5; value SW_LPO -> SW_Optical
- SW6: renamed from SWO6; value SW_LPO -> SW_Optical
- SW7: renamed from SWO7; value SW_LPO -> SW_Optical
- SW8: renamed from SWO8; value SW_LPO -> SW_Optical
- SW9: renamed from SWO9; value SW_LPO -> SW_Optical
- TP2: now in the parts list
- Y1: value 32MHz, CL12pF -> 32MHz
- Y2: value 32.768kHz, CL12.5pF -> 32.768kHz
- renumbered C12 to C21, IR1 to D1, IR10 to D10, IR11 to D11, IR12 to D12, IR13 to D13, IR14 to D14, IR15 to D15, IR16 to D16, IR17 to D17, IR18 to D18, IR19 to D19, IR2 to D2, IR20 to D20, IR21 to D21, IR22 to D22, IR23 to D23, IR24 to D24, IR25 to D25, IR26 to D26, IR27 to D27, IR28 to D28, IR29 to D29, IR3 to D3, IR30 to D30, IR31 to D31, IR32 to D32, IR33 to D33, IR34 to D34, IR35 to D35, IR36 to D36, IR37 to D37, IR38 to D38, IR39 to D39, IR4 to D4, IR40 to D40, IR41 to D41, IR42 to D42, D1 to D43, IR5 to D5, IR6 to D6, IR7 to D7, IR8 to D8, IR9 to D9, PT1 to Q1, PT10 to Q10, PT11 to Q11, PT12 to Q12, PT13 to Q13, PT14 to Q14, PT15 to Q15, PT16 to Q16, PT17 to Q17, PT18 to Q18, PT19 to Q19, PT2 to Q2, PT20 to Q20, PT21 to Q21, PT22 to Q22, PT23 to Q23, PT24 to Q24, PT25 to Q25, PT26 to Q26, PT27 to Q27, PT28 to Q28, PT29 to Q29, PT3 to Q3, PT30 to Q30, PT31 to Q31, PT32 to Q32, PT33 to Q33, PT34 to Q34, PT35 to Q35, PT36 to Q36, PT37 to Q37, PT38 to Q38, PT39 to Q39, PT4 to Q4, PT40 to Q40, PT41 to Q41, PT42 to Q42, Q1 to Q43, Q2 to Q44, Q3 to Q45, Q4 to Q46, Q5 to Q47, Q6 to Q48, Q7 to Q49, PT5 to Q5, Q8 to Q50, Q9 to Q51, Q10 to Q52, PT6 to Q6, PT7 to Q7, PT8 to Q8, PT9 to Q9, SW1 to SW43, SW2 to SW44, SW8 to SW45, SW3 to SW46, SW4 to SW47, SW6 to SW48, SW7 to SW49
Connections:
- net +3.3V: now also C25.1, C26.1
- net +5V: now also C39.2, C40.2, C41.2, C42.2, C43.2, C44.2; no longer C25.2, C26.2
- net ETA-STAT: now also TP3.1
- net GND: now also C25.2, C26.2, C39.1, C40.1, C41.1, C42.1, C43.1, C44.1; no longer C25.1, C26.1
- net key_fn3 renamed key_fn2
Other:
- moved on the sheet: AE1, BT1, C1, C11, C13, C14, C15, C16, C18, C19, C2, C20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
