File: hardware/pcb/plate/plate.kicad_sch (KiCad schematic)
At the start: 52 parts

Commit message: merge
hw:
- fix sch
- fix plate
- rename to fercus-dongle-usb-a

doc:
- add assembly
Parts:
- H1, H2, H3, H4: footprint chulaine:MountingHole_3.0mm_M3_Pad4.4mm -> chulaine:MountingHole_3.0mm_M3_Pad4.2mm
- SWH1, SWH10, SWH11, SWH12, SWH13, SWH14, SWH15, SWH16, SWH17, SWH18, SWH19, SWH2, SWH20, SWH21, SWH22, SWH23, SWH24, SWH25, SWH26, SWH27, SWH28, SWH29, SWH3, SWH30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: footprint chulaine:SW_RAESHA_Low_Profile_Optical_Plate -> chulaine:SW_RAESHA_Low_Profile_Optical_Plate_14.05mm
